Commit message: 更換原廠功能包,

File: fishbot_description/urdf/fishbot.urdf (robot description, URDF)
Before this commit: robot fishbot, 3 links, 2 joints
Links:
- added link laser_frame; visual cylinder length=0.02 radius=0.02
Joints:
- added joint laser_frame_joint: type fixed, parent base_link, child laser_frame, origin xyz=0 0 0.075 rpy=0 0 0
